Commit message: Rename files for example motor 0, joint FL_HAA

File: ros2_control_solo12/ros2_description_solo12/ros2_control/system_solo1_motor_0.ros2_control.xacro (robot description, xacro)
@@ -20,5 +20,5 @@
             <plugin>ros2_control_bolt/SystemBoltHardware</plugin>
             <param name="bolt_yaml">2.0</param>
-            <xacro:property name="prop_bolt_config_yaml" value="$(find ros2_description_solo12)/config/config_solo1.yaml" />
+            <xacro:property name="prop_bolt_config_yaml" value="$(find ros2_description_solo12)/config/config_solo1_motor_nr_0.yaml" />
             <param name="odri_config_yaml">${prop_bolt_config_yaml}</param>
             <param name="desired_starting_position">0.0 0.0 0.0 0.0 0.0 0.0</param>

File: ros2_control_solo12/ros2_description_solo12/urdf/system_solo1_motor0_description.urdf.xacro (robot description, xacro)
@@ -27,5 +27,5 @@
     </xacro:if>
   </xacro:if>
-  <xacro:include filename="$(find ros2_description_solo12)/ros2_control/system_solo1.ros2_control.xacro" />
+  <xacro:include filename="$(find ros2_description_solo12)/ros2_control/system_solo1_motor_0.ros2_control.xacro" />
   <!-- ros_control plugin for Gazebo -->
   <!-- THE PLUGIN IS MISSING -->
