Commit message: Fixed motor8 launch file errors. Got ros2 control to control motor 8

File: ros2_control_solo12/ros2_description_solo12/ros2_control/system_solo1_motor_8.ros2_control.xacro (robot description, xacro)
@@ -28,8 +28,35 @@
         </hardware>
       </xacro:unless>
-      <joint name="FL_HAA">
+      <!-- <joint name="FL_HAA">
         <command_interface name="position">
           <param name="min">-0.9</param>
           <param name="max">0.9</param>
+        </command_interface>
+        <command_interface name="velocity">
+          <param name="min">-1</param>
+          <param name="max">1</param>
+        </command_interface>
+        <command_interface name="effort">
+          <param name="min">-1</param>
+          <param name="max">1</param>
+        </command_interface>
+        <command_interface name="gain_kp">
+          <param name="min">-1000</param>
+          <param name="max">1000</param>
+        </command_interface>
+        <command_interface name="gain_kd">
+          <param name="min">-1000</param>
+          <param name="max">1000</param>
+        </command_interface>
+        <state_interface name="position"/>
+        <state_interface name="velocity"/>
+        <state_interface name="effort"/>
+        <state_interface name="gain_kp"/>
+        <state_interface name="gain_kd"/>
+      </joint> -->
+      <joint name="HL_KFE">
+        <command_interface name="position">
+          <param name="min">-2.8</param>
+          <param name="max">2.8</param>
         </command_interface>
         <command_interface name="velocity">
